Commit message: get robot loading in gazebo

File: src/simulation/descriptions/rover.world.xacro (robot description, xacro)
@@ -1,4 +1,4 @@
 <?xml version="1.0"?>
-<rover name="LUSIrover" xmlns:xacro="http://ros.org/wiki/xacro">
+<robot name="LUSIrover" xmlns:xacro="http://ros.org/wiki/xacro">
 <!-- coppied from the mutli wheel dif drive dependancy -->
     <xacro:property name="WheelSep" value="0.46"/>
@@ -13,6 +13,5 @@
         </inertial>
     </xacro:macro>
-    <link name="base_link">
-        <pose>0 0 0.1 0 0 0</pose>
+    <link name="chassis">
         <visual>
             <geometry>
@@ -25,9 +24,16 @@
             </geometry>
         </collision>
-        <xacro:default_inertial mass="15"/>
+        <xacro:default_inertial mass="14"/>
+    </link>
+    <link name="base_link">
+        <pose>0 0 0.1 0 0 0</pose>
     </link>
     <gazebo reference="base_link">
         <material>Gazebo/Blue</material>
     </gazebo>
+    <joint name="root_to_chassis" type="fixed">
+        <parent link="base_link"/>
+        <child link="chassis"/>
+    </joint>
     <!-- wheels -->
     <xacro:macro name="wheels" params = "prefex reflect">
@@ -205,3 +211,3 @@
         </plugin>
     </gazebo>
-</rover>
+</robot>

Commit message: have testing detection but camera not fully working

File: src/simulation/descriptions/rover.world.xacro (robot description, xacro)
@@ -26,4 +26,26 @@
         <xacro:default_inertial mass="14"/>
     </link>
+    <joint name="camera_joint" type="fixed">
+        <parent link="chassis"/>
+        <child link="camera_link"/>
+        <origin xyz="0.7 0.4 0" rpy="0 0 0"/>
+    </joint>
+    <link name="camera_link">
+        <visual>
+            <geometry>
+                <box size="0.010 0.03 0.03"/>
+            </geometry>
+            <material name="red"/>
+        </visual>
+    </link>
+    <gazebo reference="camera_link">
+        <material>Gazebo/Red</material>
+    </gazebo>
+    <joint name="camera_optical_joint" type="fixed">
+        <origin xyz="0 0 0" rpy="${-pi/2} 0 ${-pi/2}" />
+        <parent link="camera_link" />
+        <child link="camera_link_optical" />
+    </joint>
+    <link name="camera_link_optical"></link>
     <link name="base_link">
         <pose>0 0 0.1 0 0 0</pose>
@@ -211,3 +233,26 @@
         </plugin>
     </gazebo>
+    <gazebo reference="camera_link">
+        <material>Gazebo/Red</material>
+        <sensor name="videoStream" type="camera">
+            <pose> 0 0 0 0 0 0 </pose>
+            <visualize>true</visualize>
+            <update_rate>10</update_rate>
+            <camera>
+                <horizontal_fov>1.089</horizontal_fov>
+                <image>
+                    <format>R8G8B8</format>
+                    <width>640</width>
+                    <height>480</height>
+                </image>
+                <clip>
+                    <near>0.05</near>
+                    <far>8.0</far>
+                </clip>
+            </camera>
+            <plugin name="camera_controller" filename="libgazebo_ros_camera.so">
+                <frame_name>camera_link_optical</frame_name>
+            </plugin>
+        </sensor>
+    </gazebo>
 </robot>

Commit message: setup camera in HOOTL

File: src/simulation/descriptions/rover.world.xacro (robot description, xacro)
@@ -29,5 +29,5 @@
         <parent link="chassis"/>
         <child link="camera_link"/>
-        <origin xyz="0.7 0.4 0" rpy="0 0 0"/>
+        <origin xyz="0.4 0 0.1" rpy="0 0 0"/>
     </joint>
     <link name="camera_link">
@@ -253,4 +253,8 @@
             <plugin name="camera_controller" filename="libgazebo_ros_camera.so">
                 <frame_name>camera_link_optical</frame_name>
+                <always_on>True</always_on>
+                <updateRate>0.0</updateRate>
+                <cameraName>/LUSIrover/videoStream</cameraName>
+                <imageTopicName>/videoStream</imageTopicName>
             </plugin>
         </sensor>

Commit message: almost working 3d lusi vidsion

File: src/simulation/descriptions/rover.world.xacro (robot description, xacro)
@@ -29,5 +29,5 @@
         <parent link="chassis"/>
         <child link="camera_link"/>
-        <origin xyz="0.4 0 0.1" rpy="0 0 0"/>
+        <origin xyz="0.4 -0.1 0.1" rpy="0 0 0"/>
     </joint>
     <link name="camera_link">
@@ -48,4 +48,26 @@
     </joint>
     <link name="camera_link_optical"></link>
+    <joint name="camera2_joint" type="fixed">
+        <parent link="chassis"/>
+        <child link="camera2_link"/>
+        <origin xyz="0.4 0.1 0.1" rpy="0 0 0"/>
+    </joint>
+    <link name="camera2_link">
+        <visual>
+            <geometry>
+                <box size="0.010 0.03 0.03"/>
+            </geometry>
+            <material name="blue"/>
+        </visual>
+    </link>
+    <gazebo reference="camera2_link">
+        <material>Gazebo/Blue</material>
+    </gazebo>
+    <joint name="camera2_optical_joint" type="fixed">
+        <origin xyz="0 0 0" rpy="${-pi/2} 0 ${-pi/2}" />
+        <parent link="camera2_link" />
+        <child link="camera2_link_optical" />
+    </joint>
+    <link name="camera2_link_optical"></link>
     <link name="base_link">
         <pose>0 0 3 0 0 0</pose>
@@ -271,3 +293,30 @@
         </sensor>
     </gazebo>
+    <gazebo reference="camera2_link">
+        <material>Gazebo/Blue</material>
+        <sensor name="videoStream2" type="camera">
+            <pose> 0 0 0 0 0 0 </pose>
+            <visualize>true</visualize>
+            <update_rate>20</update_rate>
+            <camera>
+                <horizontal_fov>1.3</horizontal_fov>
+                <image>
+                    <format>R8G8B8</format>
+                    <width>640</width>
+                    <height>480</height>
+                </image>
+                <clip>
+                    <near>0.05</near>
+                    <far>8.0</far>
+                </clip>
+            </camera>
+            <plugin name="camera_controller2" filename="libgazebo_ros_camera.so">
+                <frame_name>camera_link_optical2</frame_name>
+                <always_on>True</always_on>
+                <updateRate>0.0</updateRate>
+                <cameraName>/LUSIrover/videoStream2</cameraName>
+                <imageTopicName>/videoStream2</imageTopicName>
+            </plugin>
+        </sensor>
+    </gazebo>
 </robot>

Commit message: wrist workinggit add .!

File: src/simulation/descriptions/rover.world.xacro (robot description, xacro)
@@ -29,5 +29,5 @@
         <parent link="chassis"/>
         <child link="camera_link"/>
-        <origin xyz="0.4 -0.1 0.1" rpy="0 0 0"/>
+        <origin xyz="0.4 -0.03 0.1" rpy="0 0 0"/>
     </joint>
     <link name="camera_link">
@@ -51,5 +51,5 @@
         <parent link="chassis"/>
         <child link="camera2_link"/>
-        <origin xyz="0.4 0.1 0.1" rpy="0 0 0"/>
+        <origin xyz="0.4 0.03 0.1" rpy="0 0 0"/>
     </joint>
     <link name="camera2_link">
@@ -266,5 +266,5 @@
 </plugin>
     </gazebo> -->
-    <!-- <gazebo reference="camera_link">
+    <gazebo reference="camera_link">
         <material>Gazebo/Red</material>
         <sensor name="videoStream" type="camera">
@@ -292,8 +292,8 @@
             </plugin>
         </sensor>
-    </gazebo> -->
+    </gazebo>
     <gazebo reference="camera2_link">
         <material>Gazebo/Blue</material>
-        <sensor name="videoStream" type="camera">
+        <sensor name="videoStream2" type="camera">
             <pose> 0 0 0 0 0 0 </pose>
             <visualize>true</visualize>
@@ -311,5 +311,5 @@
                 </clip>
             </camera>
-            <plugin name="camera_controller" filename="libgazebo_ros_camera.so">
+            <plugin name="camera_controller2" filename="libgazebo_ros_camera.so">
                 <frame_name>camera_link_optical</frame_name>
                 <always_on>True</always_on>
